Commit message: add joystick support in play.py; refine collision of go2.urdf to have collision that is more realistic; tron1_sf_flat implemented

File: resources/robots/go2/urdf/go2.urdf (robot description, URDF)
Before this commit: robot go2_description, 42 links, 41 joints
Links:
- link FL_hip: geometry collision cylinder length=0.12 radius=0.04; visual mesh filename=../dae/hip.dae
- link FR_hip: geometry collision cylinder length=0.12 radius=0.04; visual mesh filename=../dae/hip.dae
- link RL_hip: geometry collision cylinder length=0.12 radius=0.04; visual mesh filename=../dae/hip.dae
- link RR_hip: geometry collision cylinder length=0.12 radius=0.04; visual mesh filename=../dae/hip.dae
- link base: geometry collision box size=0.26 0.18 0.15; visual mesh filename=../dae/base.dae

Commit message: complete isaaclab integration in flat ground

File: resources/robots/go2/urdf/go2.urdf (robot description, URDF)
Before this commit: robot go2_description, 42 links, 41 joints
Links:
- link FL_calf: geometry collision cylinder length=0.12 radius=0.012; visual mesh filename=../meshes/calf.stl
- link FL_foot: geometry collision sphere radius=0.022; visual mesh filename=../meshes/foot.stl
- link FL_hip: geometry collision cylinder length=0.12 radius=0.04; visual mesh filename=../meshes/hip.stl
- link FL_thigh: geometry collision box size=0.213 0.0245 0.034; visual mesh filename=../meshes/thigh.stl
- link FR_calf: geometry collision cylinder length=0.12 radius=0.013; visual mesh filename=../meshes/calf_mirror.stl
- link FR_foot: geometry collision sphere radius=0.022; visual mesh filename=../meshes/foot.stl
- link FR_hip: geometry collision cylinder length=0.12 radius=0.04; visual mesh filename=../meshes/hip.stl
- link FR_thigh: geometry collision box size=0.213 0.0245 0.034; visual mesh filename=../meshes/thigh_mirror.stl
- link RL_calf: geometry collision cylinder length=0.12 radius=0.013; visual mesh filename=../meshes/calf.stl
- link RL_foot: geometry collision sphere radius=0.022; visual mesh filename=../meshes/foot.stl
- link RL_hip: geometry collision cylinder length=0.12 radius=0.04; visual mesh filename=../meshes/hip.stl
- link RL_thigh: geometry collision box size=0.213 0.0245 0.034; visual mesh filename=../meshes/thigh.stl
- link RR_calf: geometry collision cylinder length=0.12 radius=0.013; visual mesh filename=../meshes/calf_mirror.stl
- link RR_foot: geometry collision sphere radius=0.022; visual mesh filename=../meshes/foot.stl
- link RR_hip: geometry collision cylinder length=0.12 radius=0.04; visual mesh filename=../meshes/hip.stl
- link RR_thigh: geometry collision box size=0.213 0.0245 0.034; visual mesh filename=../meshes/thigh_mirror.stl
- link base: geometry collision box size=0.26 0.18 0.15; visual mesh filename=../meshes/base.stl
